File: PE42424A/PE42424A.kicad_pcb (KiCad board)
At the start: 2 copper layers, 1 x 13.7 mm, 4 parts

Commit message: added switches
Other:
- board size 1 x 13.7 mm -> 16.9 x 17.9 mm
Changed lines of the file:
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@@
     (pad_to_mask_clearance 0)
     (pcbplotparams
-      (layerselection 0x00010fc_ffffffff)
+      (layerselection 0x00010cc_ffffffff)
       (plot_on_all_layers_selection 0x0000000_00000000)
       (disableapertmacros false)
@@
       (outputformat 1)
       (mirror false)
-      (drillshape 1)
+      (drillshape 0)
       (scaleselection 1)
-      (outputdirectory "")
+      (outputdirectory "/Volumes/mic FD/RF/PE42424A/")
     )
   )
@@
   (gr_circle (center 111.5 77.82) (end 112 77.82)
     (stroke (width 0.01) (type default)) (fill none) (layer "Edge.Cuts"))
+  (gr_rect (start 102.4 67.7) (end 119.3 85.6)
+    (stroke (width 0.1) (type default)) (fill none) (layer "Edge.Cuts"))
   (gr_circle (center 111.5 75.28) (end 112 75.28)
     (stroke (width 0.01) (type default)) (fill none) (layer "Edge.Cuts"))
